Commit message: rviz mod

File: src/robot_description/urdf/2wheel.xacro (robot description, xacro)
@@ -69,4 +69,5 @@
    </gazebo>
 <!-- End: For URDF to Gazebo compatibility -->
+	<link name="dummy_link"/>
   <link name="link_chassis">
     <!-- pose and inertial -->
@@ -92,4 +93,9 @@
     </visual>
   </link>
+	<joint name="Base" type="fixed">
+    <origin rpy="0 0 0" xyz="0 0 0"/>
+		<child link="link_chassis"/>
+    <parent link="dummy_link"/>
+  </joint>
   <link name="link_left_wheel">
     <inertial>

Commit message: Imu test and first empirical controller.

File: src/robot_description/urdf/2wheel.xacro (robot description, xacro)
@@ -54,5 +54,6 @@
       <plugin name="imu_plugin" filename="libgazebo_ros_imu.so">
           <alwaysOn>true</alwaysOn>
-          <bodyName>link_chassis</bodyName>
+					<updateRate>50</updateRate>
+          <bodyName>imu_link</bodyName>
           <topicName>imu</topicName>
           <serviceName>imu_service</serviceName>
@@ -70,4 +71,5 @@
 <!-- End: For URDF to Gazebo compatibility -->
 	<link name="dummy_link"/>
+	<link name="imu_link"/>
   <link name="link_chassis">
     <!-- pose and inertial -->
@@ -97,4 +99,9 @@
 		<child link="link_chassis"/>
     <parent link="dummy_link"/>
+  </joint>
+	<joint name="Imu" type="fixed">
+    <origin rpy="0 0 0" xyz="0 0 0.3"/>
+		<child link="imu_link"/>
+    <parent link="link_chassis"/>
   </joint>
   <link name="link_left_wheel">

Commit message: IMU sensor simulation in progress. Further inspection needed.

File: src/robot_description/urdf/2wheel.xacro (robot description, xacro)
@@ -35,4 +35,27 @@
     <material>Gazebo/Red</material>
   </gazebo>
+<!--
+	<gazebo reference="imu_link">
+    <gravity>true</gravity>
+    <sensor name="imu_sensor" type="imu">
+      <always_on>true</always_on>
+      <update_rate>100</update_rate>
+      <visualize>true</visualize>
+      <topic>__default_topic__</topic>
+			<imu/>
+      <plugin filename="libgazebo_ros_imu_sensor.so" name="imu_plugin">
+        <topicName>imu</topicName>
+        <bodyName>imu_link</bodyName>
+        <updateRateHZ>10.0</updateRateHZ>
+        <gaussianNoise>0.0</gaussianNoise>
+        <xyzOffset>0 0 0</xyzOffset>
+        <rpyOffset>0 0 0</rpyOffset>
+        <frameName>imu_link</frameName>
+        <initialOrientationAsReference>false</initialOrientationAsReference>
+      </plugin>
+      <pose>0 0 0 0 0 0</pose>
+    </sensor>
+  </gazebo>
+-->
   <gazebo>
     <plugin filename="libgazebo_ros_diff_drive.so" name="differential_drive_controller">
@@ -51,13 +74,15 @@
     </plugin>
   </gazebo>
+	<!-- -->
   <gazebo>
       <plugin name="imu_plugin" filename="libgazebo_ros_imu.so">
           <alwaysOn>true</alwaysOn>
-					<updateRate>50</updateRate>
-          <bodyName>imu_link</bodyName>
+					<updateRate>100</updateRate>
+          <bodyName>dummy_link</bodyName>
           <topicName>imu</topicName>
           <serviceName>imu_service</serviceName>
           <gaussianNoise>0.0</gaussianNoise>
           <rpyOffsets>0 0 0</rpyOffsets>
+					<xyzOffset>0 0 0.3</xyzOffset>
           <accelDrift>0.5 0.5 0.5</accelDrift>
           <accelGaussianNoise>0.35 0.35 0.3</accelGaussianNoise>
@@ -66,10 +91,16 @@
           <headingDrift>0.0</headingDrift>
           <headingGaussianNoise>0.00</headingGaussianNoise>
-          <updateRate>00</updateRate>
       </plugin>
    </gazebo>
+<!-- xyzOffset is a workaround for problem. check generated code with gz sdf -p 2wheel.xacro-->
 <!-- End: For URDF to Gazebo compatibility -->
 	<link name="dummy_link"/>
-	<link name="imu_link"/>
+	<link name="imu_link">
+    <inertial>
+      <mass value="0.0001"/>
+      <origin rpy="0 0 0" xyz="0 0 0"/>
+      <inertia ixx="0.000001" ixy="0" ixz="0" iyy="0.000001" iyz="0" izz="0.000001"/>
+    </inertial>
+  </link>
   <link name="link_chassis">
     <!-- pose and inertial -->
@@ -95,10 +126,10 @@
     </visual>
   </link>
-	<joint name="Base" type="fixed">
+	<joint name="base_joint" type="fixed">
     <origin rpy="0 0 0" xyz="0 0 0"/>
 		<child link="link_chassis"/>
     <parent link="dummy_link"/>
   </joint>
-	<joint name="Imu" type="fixed">
+	<joint name="imu_joint" type="fixed">
     <origin rpy="0 0 0" xyz="0 0 0.3"/>
 		<child link="imu_link"/>

Commit message: Added "Tablon" visual

File: src/robot_description/urdf/2wheel.xacro (robot description, xacro)
@@ -25,7 +25,16 @@
     <color rgba="1.0 1.0 1.0 1.0"/>
   </material>
+  <material name="plank">
+    <color rgba="0.9098 0.77255 0.2314 1.0"/>
+  </material>
 <!-- Start: For URDF to Gazebo compatibility -->
   <gazebo reference="link_chassis">
-    <material>Gazebo/Black</material>
+    <material>Gazebo/Yellow</material>
+  </gazebo>
+  <gazebo reference="link_mouth">
+    <material>Gazebo/Blue</material>
+  </gazebo>
+  <gazebo reference="link_eyes">
+    <material>Gazebo/Red</material>
   </gazebo>
   <gazebo reference="link_left_wheel">
@@ -119,9 +128,47 @@
     </collision>
     <visual>
-      <origin rpy="0 0 0" xyz="0 0 0.3"/>
-      <geometry>
-        <box size="0.1 0.3 0.6"/>
-      </geometry>
-      <material name="black"/>
+      <!-- <origin rpy="0 0 0" xyz="0 0 0.3"/> -->
+			<origin rpy="0 0 0" xyz="0 0 0"/>
+      <geometry>
+        <!-- <box size="0.1 0.3 0.6"/> -->
+				<mesh filename="package://robot_description/stl/Plank.stl" scale="1 1 1"/>
+      </geometry>
+      <material name="plank"/>
+    </visual>
+  </link>
+	<link name="link_mouth">
+    <!-- pose and inertial -->
+    <pose>0 0 0.1 0 0 0</pose>
+    <inertial>
+      <mass value="0.0001"/>
+      <origin rpy="0 0 0" xyz="0 0 0"/>
+      <inertia ixx="0.000001" ixy="0" ixz="0" iyy="0.000001" iyz="0" izz="0.000001"/>
+    </inertial>
+    <visual>
+      <!-- <origin rpy="0 0 0" xyz="0 0 0.3"/> -->
+			<origin rpy="0 0 0" xyz="0 0 0"/>
+      <geometry>
+        <!-- <box size="0.1 0.3 0.6"/> -->
+				<mesh filename="package://robot_description/stl/mouth.stl" scale="1 1 1"/>
+      </geometry>
+      <material name="blue"/>
+    </visual>
+  </link>
+	<link name="link_eyes">
+    <!-- pose and inertial -->
+    <pose>0 0 0.1 0 0 0</pose>
+    <inertial>
+      <mass value="0.0001"/>
+      <origin rpy="0 0 0" xyz="0 0 0"/>
+      <inertia ixx="0.000001" ixy="0" ixz="0" iyy="0.000001" iyz="0" izz="0.000001"/>
+    </inertial>
+    <visual>
+      <!-- <origin rpy="0 0 0" xyz="0 0 0.3"/> -->
+			<origin rpy="0 0 0" xyz="0 0 0"/>
+      <geometry>
+        <!-- <box size="0.1 0.3 0.6"/> -->
+				<mesh filename="package://robot_description/stl/eyes.stl" scale="1 1 1"/>
+      </geometry>
+      <material name="red"/>
     </visual>
   </link>
@@ -136,4 +183,14 @@
     <parent link="link_chassis"/>
   </joint>
+	<joint name="eyes_joint" type="fixed">
+    <origin rpy="0 0 0" xyz="0 0 0"/>
+		<child link="link_eyes"/>
+    <parent link="link_chassis"/>
+  </joint>
+	<joint name="mouth_joint" type="fixed">
+    <origin rpy="0 0 0" xyz="0 0 0"/>
+		<child link="link_mouth"/>
+    <parent link="link_chassis"/>
+  </joint>
   <link name="link_left_wheel">
     <inertial>

Commit message: Added new model related to real protoype.

File: src/robot_description/urdf/2wheel.xacro (robot description, xacro)
@@ -11,5 +11,5 @@
   </material>
   <material name="grey">
-    <color rgba="0.2 0.2 0.2 1.0"/>
+    <color rgba="0.6 0.6 0.6 1.0"/>
   </material>
   <material name="orange">
@@ -29,18 +29,24 @@
   </material>
 <!-- Start: For URDF to Gazebo compatibility -->
+	<!-- LINKS -->
   <gazebo reference="link_chassis">
-    <material>Gazebo/Yellow</material>
-  </gazebo>
-  <gazebo reference="link_mouth">
-    <material>Gazebo/Blue</material>
-  </gazebo>
-  <gazebo reference="link_eyes">
-    <material>Gazebo/Red</material>
+    <material>Gazebo/Grey</material>
   </gazebo>
   <gazebo reference="link_left_wheel">
-    <material>Gazebo/Red</material>
+    <material>Gazebo/Black</material>
+    <mu1>0.4</mu1>
+    <mu2>0.4</mu2>
   </gazebo>
   <gazebo reference="link_right_wheel">
-    <material>Gazebo/Red</material>
+    <material>Gazebo/Black</material>
+    <mu1>0.4</mu1>
+    <mu2>0.4</mu2>
+  </gazebo>
+	<!-- JOINTS -->
+  <gazebo reference="joint_right_wheel">
+		<!-- <gearbox_ratio>0.0294</gearbox_ratio> -->
+  </gazebo>
+  <gazebo reference="joint_left_wheel">
+		<!-- <gearbox_ratio>0.0294</gearbox_ratio> -->
   </gazebo>
 <!--
@@ -67,4 +73,5 @@
   </gazebo>
 -->
+	<!-- PLUGINS -->
   <gazebo>
     <plugin filename="libgazebo_ros_diff_drive.so" name="differential_drive_controller">
@@ -74,7 +81,7 @@
       <leftJoint>joint_left_wheel</leftJoint>
       <rightJoint>joint_right_wheel</rightJoint>
-      <wheelSeparation>0.34</wheelSeparation>
-      <wheelDiameter>0.2</wheelDiameter>
-      <torque>10</torque>
+      <wheelSeparation>0.134418</wheelSeparation>
+      <wheelDiameter>0.07</wheelDiameter>
+      <wheelTorque>0.8</wheelTorque>
       <commandTopic>cmd_vel</commandTopic>
       <odometryTopic>odom</odometryTopic>
@@ -93,5 +100,5 @@
           <gaussianNoise>0.0</gaussianNoise>
           <rpyOffsets>0 0 0</rpyOffsets>
-					<xyzOffset>0 0 0.3</xyzOffset>
+					<xyzOffset>0 0 0.0434</xyzOffset>
           <accelDrift>0.5 0.5 0.5</accelDrift>
           <accelGaussianNoise>0.35 0.35 0.3</accelGaussianNoise>
@@ -114,15 +121,15 @@
   <link name="link_chassis">
     <!-- pose and inertial -->
-    <pose>0 0 0.1 0 0 0</pose>
-    <inertial>
-      <mass value="2"/>
-      <origin rpy="0 0 0" xyz="0 0 0.3"/>
-      <inertia ixx="0.075" ixy="0" ixz="0" iyy="0.061667" iyz="0" izz="0.01667"/>
+    <pose>0 0 0.25 0 0 0</pose>
+    <inertial>
+      <mass value="0.8369"/>
+      <origin rpy="0 0 0" xyz="-0.000631 0.000044 0.016159"/>
+      <inertia ixx="6.495E-3" ixy="979.958E-9" ixz="-1.335E-5" iyy=" 2.282E-3" iyz="1000.67e-9" izz="5.266E-3"/>
     </inertial>
     <!-- body -->
     <collision name="collision_chassis">
-      <origin rpy="0 0 0" xyz="0 0 0.3"/>
-      <geometry>
-        <box size="0.1 0.3 0.6"/>
+      <origin rpy="0 0 0" xyz="0 0 0.0434"/>
+      <geometry>
+        <box size="0.10311 0.200188 0.166021"/>
       </geometry>
     </collision>
@@ -132,43 +139,7 @@
       <geometry>
         <!-- <box size="0.1 0.3 0.6"/> -->
-				<mesh filename="package://robot_description/stl/Plank.stl" scale="1 1 1"/>
-      </geometry>
-      <material name="plank"/>
-    </visual>
-  </link>
-	<link name="link_mouth">
-    <!-- pose and inertial -->
-    <pose>0 0 0.1 0 0 0</pose>
-    <inertial>
-      <mass value="0.0001"/>
-      <origin rpy="0 0 0" xyz="0 0 0"/>
-      <inertia ixx="0.000001" ixy="0" ixz="0" iyy="0.000001" iyz="0" izz="0.000001"/>
-    </inertial>
-    <visual>
-      <!-- <origin rpy="0 0 0" xyz="0 0 0.3"/> -->
-			<origin rpy="0 0 0" xyz="0 0 0"/>
-      <geometry>
-        <!-- <box size="0.1 0.3 0.6"/> -->
-				<mesh filename="package://robot_description/stl/mouth.stl" scale="1 1 1"/>
-      </geometry>
-      <material name="blue"/>
-    </visual>
-  </link>
-	<link name="link_eyes">
-    <!-- pose and inertial -->
-    <pose>0 0 0.1 0 0 0</pose>
-    <inertial>
-      <mass value="0.0001"/>
-      <origin rpy="0 0 0" xyz="0 0 0"/>
-      <inertia ixx="0.000001" ixy="0" ixz="0" iyy="0.000001" iyz="0" izz="0.000001"/>
-    </inertial>
-    <visual>
-      <!-- <origin rpy="0 0 0" xyz="0 0 0.3"/> -->
-			<origin rpy="0 0 0" xyz="0 0 0"/>
-      <geometry>
-        <!-- <box size="0.1 0.3 0.6"/> -->
-				<mesh filename="package://robot_description/stl/eyes.stl" scale="1 1 1"/>
-      </geometry>
-      <material name="red"/>
+				<mesh filename="package://robot_description/stl/Real/Base.stl" scale="0.001 0.001 0.001"/>
+      </geometry>
+      <material name="grey"/>
     </visual>
   </link>
@@ -179,71 +150,70 @@
   </joint>
 	<joint name="imu_joint" type="fixed">
-    <origin rpy="0 0 0" xyz="0 0 0.3"/>
+    <origin rpy="0 0 0" xyz="0 0 0.0434"/>
 		<child link="imu_link"/>
     <parent link="link_chassis"/>
   </joint>
-	<joint name="eyes_joint" type="fixed">
-    <origin rpy="0 0 0" xyz="0 0 0"/>
-		<child link="link_eyes"/>
-    <parent link="link_chassis"/>
-  </joint>
-	<joint name="mouth_joint" type="fixed">
-    <origin rpy="0 0 0" xyz="0 0 0"/>
-		<child link="link_mouth"/>
-    <parent link="link_chassis"/>
-  </joint>
   <link name="link_left_wheel">
     <inertial>
-      <mass value="0.2"/>
-      <origin rpy="0 1.5707 1.5707" xyz="0 0 0"/>
-      <inertia ixx="0.001" ixy="0" ixz="0" iyy="0.0005" iyz="0" izz="0.0005"/>
+      <mass value="0.087306"/>
+      <origin rpy="0 0 0" xyz="0 -0.38566 0"/>
+      <inertia ixx="2.776E-5" ixy="15.762E-9" ixz="-0.097E-9" iyy="4.868E-5" iyz="-0.371E-9" izz="2.774E-5"/>
     </inertial>
     <collision name="link_left_wheel_collision">
-      <origin rpy="0 1.5707 1.5707" xyz="0 0 0"/>
-      <geometry>
-        <cylinder length="0.04" radius="0.1"/>
+      <origin rpy="0 1.5707 1.5707" xyz="0 0.01205 0"/>
+      <geometry>
+        <cylinder length="0.0241" radius="0.035"/>
       </geometry>
     </collision>
     <visual name="link_left_wheel_visual">
-      <origin rpy="0 1.5707 1.5707" xyz="0 0 0"/>
-      <geometry>
-        <cylinder length="0.04" radius="0.1"/>
-      </geometry>
+      <origin rpy="0 0 3.1415927" xyz="0 0 0"/>
+      <geometry>
+        <!-- <box size="0.1 0.3 0.6"/> -->
+				<mesh filename="package://robot_description/stl/Real/Wheel.stl" scale="0.001 0.001 0.001"/>
+      </geometry>
+      <material name="grey"/>
     </visual>
   </link>
-  <joint name="joint_left_wheel" type="continuous">
-    <origin rpy="0 0 0" xyz="0 0.17 0"/>
+  <joint name="joint_left_wheel" type="revolute">  <!-- We set revolute with infinite limits as a workaround to sdf conversion problems -->
+    <origin rpy="0 0 0" xyz="-0.000944 0.110418 -0.027797"/>
     <child link="link_left_wheel"/>
     <parent link="link_chassis"/>
     <axis rpy="0 0 0" xyz="0 1 0"/>
-    <limit effort="10000" velocity="1000"/>
-    <joint_properties damping="1.0" friction="1.0"/>
+		<limit effort="0.8" velocity="30" lower="-1e+16" upper="1e+16" />
+    <!--<limit effort="0.8" velocity="30"/>-->
+    <dynamics damping="0.0005" friction="0.0005"/>  <!-- damping coefficient: [N*m*s/rad] 0.0005-->
+		<safety_controller k_velocity="0.026"/>  <!-- Kv en este caso: Torque/vel (http://wiki.ros.org/pr2_controller_manager/safety_limits) -->
   </joint>
   <link name="link_right_wheel">
     <inertial>
-      <mass value="0.2"/>
-      <origin rpy="0 1.5707 1.5707" xyz="0 0 0"/>
-      <inertia ixx="0.001" ixy="0" ixz="0" iyy="0.0005" iyz="0" izz="0.0005"/>
+      <mass value="0.087306"/>
+      <origin rpy="0 0 0" xyz="0 +0.38566 0"/>
+      <inertia ixx="2.776E-5" ixy="15.762E-9" ixz="-0.097E-9" iyy="4.868E-5" iyz="0.371E-9" izz="2.774E-5"/>
     </inertial>
     <collision name="link_right_wheel_collision">
-      <origin rpy="0 1.5707 1.5707" xyz="0 0 0"/>
-      <geometry>
-        <cylinder length="0.04" radius="0.1"/>
+      <origin rpy="0 1.5707 1.5707" xyz="0 -0.01205 0"/>
+      <geometry>
+        <cylinder length="0.0241" radius="0.035"/>
       </geometry>
     </collision>
     <visual name="link_right_wheel_visual">
-      <origin rpy="0 1.5707 1.5707" xyz="0 0 0"/>
-      <geometry>
-        <cylinder length="0.04" radius="0.1"/>
-      </geometry>
+      <origin rpy="0 0 0" xyz="0 0 0"/>
+      <geometry>
+        <!-- <box size="0.1 0.3 0.6"/> -->
+				<mesh filename="package://robot_description/stl/Real/Wheel.stl" scale="0.001 0.001 0.001"/>
+      </geometry>
+      <material name="grey"/>
     </visual>
   </link>
-  <joint name="joint_right_wheel" type="continuous">
-    <origin rpy="0 0 0" xyz="0 -0.17 0"/>
+  <joint name="joint_right_wheel" type="revolute">  <!-- We set revolute with infinite limits as a workaround to sdf conversion problems -->
+    <origin rpy="0 0 0" xyz="-0.000944 -0.110418 -0.027797"/>
     <child link="link_right_wheel"/>
     <parent link="link_chassis"/>
     <axis rpy="0 0 0" xyz="0 1 0"/>
-    <limit effort="10000" velocity="1000"/>
-    <joint_properties damping="1.0" friction="1.0"/>
-  </joint>
+		<limit effort="0.8" velocity="30" lower="-1e+16" upper="1e+16" />
+    <!--<limit effort="0.8" velocity="30"/>-->
+  	<dynamics damping="0.0005" friction="0.0005"/>  <!-- damping coefficient: [N*m*s/rad] -->
+		<safety_controller k_velocity="0.026"/>  <!-- Kv en este caso: Torque/vel (http://wiki.ros.org/pr2_controller_manager/safety_limits) -->
+  </joint>
+	<!-- TRANSMISION (TODO)-->
 </robot>
